File: KiCAD/Latch colis/Latch colis.kicad_sch (KiCad schematic)
At the start: 12 parts, among them J1 KF301-2P, J2 KF301-2P, J3 KF301-2P, J4 Jauges, K1 Relay_SPDT, K2 Relay_SPDT, Q1 2N2222A, U1 Heltec_LoRa32_V2_RST_side, U2 Module HX711

Commit message: Fusion boite-aux-lettres-lora : ajout docs, photos, variantes KiCad, binaires de test
- Docs/ : plan cotes boîte aux lettres, pinout Heltec, datasheet jauge 50kg, référence latch
- KiCAD : 4 variantes schémas latch MOSFET (v1, NE555, avec_lora, RS) + images références
- KiCAD Latch colis : fichiers PCB/SCH mis à jour (09-11/09), gravure actualisée
- KiCAD Symboles : bibliothèque Heltec LoRa32 V2
- src/bin : emetteur_test_1s, recepteur_test_1s, test_hx711
- src/archive : historique des premières versions emetteur/recepteur
- html/ : calculateurs (circuit verrouillage, échelle dBm, ping vs reçus)
- Lightburn : fichiers gravure laser (.lbrn2, .cwprj)
- .cargo/config.toml : target-dir + CARGO_WORKSPACE_DIR (fix embuild remote_component)
- Boîte aux lettres.md : documentation technique projet

Co-Authored-By: Claude Sonnet 4.6 <noreply@anthropic.com>
Parts:
- Q1: footprint Package_TO_SOT_THT:TO-92L_Inline_Wide -> Package_TO_SOT_THT:TO-92
Other:
- title: Gestion courrier boîtes aux lettres -> Gestion courriers boîtes aux lettres
Changed lines of the file:
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@@
 	(paper "A4")
 	(title_block
-		(title "Gestion courrier boîtes aux lettres")
+		(title "Gestion courriers boîtes aux lettres")
 		(date "2026-09-06")
 	)
@@
 			)
 		)
-		(property "Footprint" "Package_TO_SOT_THT:TO-92L_Inline_Wide"
+		(property "Footprint" "Package_TO_SOT_THT:TO-92"
 			(at 190.5 92.71 0)
 			(hide yes)
