File: KiCAD/Latch colis/Latch colis sans inter/Latch colis sans inter.kicad_pcb (KiCad board)
At the start: 2 copper layers, 80.5 x 56 mm, 8 parts, among them J1 KF301-2P, J4 Jauges, Q1 2N2222A, Q2 BS250, U1 Heltec_LoRa32_V2_RST_side, U2 Module HX711

Commit message: Synchro fichiers Wi-Fi/NTP/correction d'horloge depuis C:\rust
Co-Authored-By: Claude Sonnet 5 <noreply@anthropic.com>
Parts:
- J4: footprint Connector_PinHeader_2.54mm:PinHeader_1x06_P2.54mm_Vertical -> Connector_PinHeader_2.54mm:PinHeader_1x04_P2.54mm_Vertical
- moved R1 0.51 mm to (92.0, 57.8)
Routing:
- net Net-(J4-Pin_6): track 9.31 -> 0.00 mm
- net Net-(J4-Pin_5): track 9.39 -> 0.12 mm
- net Net-(U1-33): track 11.3 -> 11.9 mm
Changed lines of the file:
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@@
 	(footprint "Resistor_THT:R_Axial_DIN0207_L6.3mm_D2.5mm_P10.16mm_Horizontal"
 		(layer "F.Cu")
-		(at 92.5 57.84 -90)
+		(at 92 57.75 -90)
 		(descr "Resistor, Axial_DIN0207 series, Axial, Horizontal, pin pitch=10.16mm, 0.25W = 1/4W, length*diameter=6.3*2.5mm^2, http://cdn-reichelt.de/documents/datenblatt/B400/1_4W%23YAG.pdf")
 		(tags "Resistor Axial_DIN0207 series Axial Horizontal pin pitch 10.16mm 0.25W = 1/4W length 6.3mm diameter 2.5mm")
@@
 		)
 	)
-	(footprint "Connector_PinHeader_2.54mm:PinHeader_1x06_P2.54mm_Vertical"
+	(footprint "Connector_PinHeader_2.54mm:PinHeader_1x04_P2.54mm_Vertical"
 		(layer "F.Cu")
 		(at 133.5 50.5)
-		(descr "Through hole straight pin header, 1x06, 2.54mm pitch, single row")
-		(tags "Through hole pin header THT 1x06 2.54mm single row")
+		(descr "Through hole straight pin header, 1x04, 2.54mm pitch, single row")
+		(tags "Through hole pin header THT 1x04 2.54mm single row")
 		(property "Reference" "J4"
 			(at 0 -2.38 0)
@@
 		)
 		(property "Value" "Jauges"
-			(at 0 15.08 0)
+			(at 0 10 0)
 			(layer "F.Fab")
 			(effects
@@
 		(fp_line
 			(start -1.38 1.27)
-			(end -1.38 14.08)
+			(end -1.38 9)
 			(stroke
 				(width 0.12)
@@
 		)
 		(fp_line
-			(start -1.38 14.08)
-			(end 1.38 14.08)
+			(start -1.38 9)
+			(end 1.38 9)
 			(stroke
 				(width 0.12)
@@
 		(fp_line
 			(start 1.38 1.27)
-			(end 1.38 14.08)
+			(end 1.38 9)
 			(stroke
 				(width 0.12)
@@
 		(fp_rect
 			(start -1.77 -1.77)
-			(end 1.77 14.47)
+			(end 1.77 9.39)
 			(stroke
 				(width 0.05)
@@
 		)
 		(fp_line
-			(start -1.27 13.97)
+			(start -1.27 8.89)
 			(end -1.27 -0.635)
 			(stroke
@@
 		(fp_line
 			(start 1.27 -1.27)
-			(end 1.27 13.97)
-			(stroke
-				(width 0.1)
-				(type solid)
-			)
-			(layer "F.Fab")
-		)
-		(fp_line
-			(start 1.27 13.97)
-			(end -1.27 13.97)
+			(end 1.27 8.89)
+			(stroke
+				(width 0.1)
+				(type solid)
+			)
+			(layer "F.Fab")
+		)
+		(fp_line
+			(start 1.27 8.89)
+			(end -1.27 8.89)
 			(stroke
 				(width 0.1)
@@
 		)
 		(fp_text user "${REFERENCE}"
-			(at 0 6.35 90)
+			(at 0 3.81 90)
 			(layer "F.Fab")
 			(effects
@@
 			(pintype "passive")
 		)
-		(pad "5" thru_hole circle
-			(at 0 10.16)
-			(size 1.7 1.7)
-			(drill 1)
-			(layers "*.Cu" "*.Mask")
-			(remove_unused_layers no)
-			(net "Net-(J4-Pin_5)")
-			(pinfunction "Pin_5_5")
-			(pintype "passive")
-		)
-		(pad "6" thru_hole circle
-			(at 0 12.7)
-			(size 1.7 1.7)
-			(drill 1)
-			(layers "*.Cu" "*.Mask")
-			(remove_unused_layers no)
-			(net "Net-(J4-Pin_6)")
-			(pinfunction "Pin_6_6")
-			(pintype "passive")
-		)
 		(embedded_fonts no)
-		(model "${KICAD10_3DMODEL_DIR}/Connector_PinHeader_2.54mm.3dshapes/PinHeader_1x06_P2.54mm_Vertical.step"
+		(model "${KICAD10_3DMODEL_DIR}/Connector_PinHeader_2.54mm.3dshapes/PinHeader_1x04_P2.54mm_Vertical.step"
 			(offset
 				(xyz 0 0 0)
@@
 	)
 	(segment
-		(start 92.5 56.5)
-		(end 92.5 57.84)
+		(start 89.46 53.46)
+		(end 92.1 56.1)
 		(width 1)
 		(layer "F.Cu")
@@
 	)
 	(segment
-		(start 89.46 53.46)
-		(end 92.5 56.5)
+		(start 92.1 56.1)
+		(end 92.1 57.65)
+		(width 1)
+		(layer "F.Cu")
+		(net "Net-(Q1-Pad2)")
+	)
+	(segment
+		(start 92.1 57.65)
+		(end 92 57.75)
 		(width 1)
 		(layer "F.Cu")
@@
 	)
 	(segment
-		(start 92.5 68)
-		(end 99.5 68)
-		(width 1)
-		(layer "F.Cu")
-		(net "Net-(U1-33)")
-	)
-	(segment
 		(start 99.5 68)
 		(end 101.31 69.81)
@@
 	)
 	(segment
+		(start 92 67.91)
+		(end 92.09 68)
+		(width 1)
+		(layer "F.Cu")
+		(net "Net-(U1-33)")
+	)
+	(segment
+		(start 92.09 68)
+		(end 99.5 68)
+		(width 1)
+		(layer "F.Cu")
+		(net "Net-(U1-33)")
+	)
+	(segment
 		(start 86.5 61)
 		(end 86.5 63)
@@
 	)
 	(segment
-		(start 124.37 61)
-		(end 133.16 61)
-		(width 1)
-		(layer "F.Cu")
-		(net "Net-(J4-Pin_5)")
-	)
-	(segment
 		(start 124.285 61.085)
 		(end 124.37 61)
@@
 	)
 	(segment
-		(start 133.16 61)
-		(end 133.5 60.66)
-		(width 1)
-		(layer "F.Cu")
-		(net "Net-(J4-Pin_5)")
-	)
-	(segment
-		(start 133.195 63.505)
-		(end 133.5 63.2)
-		(width 1)
-		(layer "F.Cu")
-		(net "Net-(J4-Pin_6)")
-	)
-	(segment
-		(start 124.315 63.505)
-		(end 133.195 63.505)
-		(width 1)
-		(layer "F.Cu")
-		(net "Net-(J4-Pin_6)")
-	)
-	(segment
